File: BrainA1-6Mar2015.brd (EAGLE design)
At the start: 81.4 x 53.3 mm, 139 parts, among them IC1 OP2177ARMZ, IC2 OPA2111KP, IC3 OP4177ARZ, IC4 OPA2111KP, IC5 TLC555CDR, IC6 TAR5SB50, IC7 LT1761ES5-5, K1 AQY221R2VY, K2 AQY221R2VY

Commit message: v0.2
update
Parts:
- added SJ17, SJ6: (no value), jumper:SJ
- moved JP2 19.6 mm to (13.9, 47.8)
- moved JP1 19.5 mm to (13.9, 45.2)
- moved JP3 4.92 mm to (13.9, 23.8)
- moved JP4 4.92 mm to (13.9, 26.3)
- moved R24 1.50 mm to (16.9, 45.1)
- moved C28 1.20 mm to (19.6, 45.1)
- moved R27 1.10 mm to (19.4, 41.7)
- moved R11 0.60 mm to (17.9, 50.5)
- moved R12 0.60 mm to (17.9, 48.2)
Connections:
- net N$28: now also SJ17.2
- net N$52: now also SJ6.2
- net N$77: now also SJ6.1
- net N$81: now also SJ17.1
Routing:
- net N$52: track 26.9 -> 12.0 mm
- net N$81: track 10.6 -> 23.3 mm
- net N$77: track 15.8 -> 19.3 mm
- net N$13: track 33.2 -> 30.0 mm
- net N$37: track 16.1 -> 13.2 mm
- net N$55: track 30.5 -> 27.8 mm
- net N$24: track 25.6 -> 24.2 mm
- net N$6: track 19.0 -> 17.9 mm
- net GND: track 522.5 -> 523.5 mm
- net N$28: track 19.5 -> 20.1 mm
- net N$22: track 26.7 -> 26.1 mm
