File: BrainA1-11March2015.brd (EAGLE design)
At the start: 81.4 x 53.3 mm, 141 parts, among them IC1 OP2177ARMZ, IC2 OPA2111KP, IC3 OP4177ARZ, IC4 OPA2111KP, IC5 TLC555CDR, IC6 TAR5SB50, IC7 LT1761ES5-5, K1 AQY221R2VY, K2 AQY221R2VY

Commit message: V0.2
update
Parts:
- removed JP1, JP2, JP3, JP4: (no value), pinhead:1X01
- removed LR-IN1: (no value), pinhead:2X03/90
- added JP5: (no value), pinhead:2X05/90
- moved SJ6 15.5 mm to (17.4, 26.9), turned to 180 degrees
- moved SJ17 12.9 mm to (17.4, 41.9), turned to 180 degrees
- moved R28 4.33 mm to (17.2, 24.2), turned to 180 degrees
- moved R27 3.55 mm to (21.2, 44.7)
- moved R24 2.70 mm to (14.2, 45.1)
- moved C28 2.40 mm to (17.1, 45.1)
- moved R14 1.87 mm to (17.2, 21.8), turned to 0 degrees
- moved C19 0.58 mm to (17.2, 19.0), turned to 0 degrees
Connections:
- removed net LR-IN: LR-IN1.2, R14.1
- new net N$114: JP5.4, R14.1
- net GND: now also JP5.5, JP5.6; no longer LR-IN1.3, LR-IN1.4
- net N$28: now also JP5.10, JP5.8; no longer JP4.1, LR-IN1.6
- net N$37: now also JP5.7; no longer LR-IN1.5
- net N$52: now also JP5.2; no longer JP2.1
- net N$77: now also JP5.1, JP5.3; no longer JP1.1, LR-IN1.1
- net N$81: now also JP5.9; no longer JP3.1
Routing:
- net GND: track 523.5 -> 494.7 mm, vias 14 -> 13
- net N$52: track 12.0 -> 30.1 mm
- net N$81: track 23.3 -> 41.0 mm, vias 0 -> 1
- net N$28: track 20.1 -> 5.18 mm
- net N$77: track 19.3 -> 5.16 mm
- net N$114: track 0.00 -> 12.4 mm, vias 0 -> 1
- net LR-IN: track 9.82 -> 0.00 mm
- net N$13: track 30.0 -> 34.0 mm
- net N$37: track 13.2 -> 17.2 mm
- net N$24: track 24.2 -> 26.7 mm
- net N$40: track 25.9 -> 28.3 mm
- net N$6: track 17.9 -> 16.2 mm
- net N$42: track 21.3 -> 22.9 mm
