File: BrainA1-11March2015.sch (EAGLE design)
At the start: 141 parts, among them IC1 OP2177ARMZ, IC2 OPA2111KP, IC3 OP4177ARZ, IC4 OPA2111KP, IC5 TLC555CDR, IC6 TAR5SB50, IC7 LT1761ES5-5, K1 AQY221R2VY, K2 AQY221R2VY

Commit message: V0.2
update
Parts:
- removed JP1, JP2, JP3, JP4: (no value), pinhead:PINHD-1X1
- removed LR-IN1: (no value), pinhead:PINHD-2X3/90
- added JP5: (no value), pinhead:PINHD-2X5/90
Connections:
- removed net LR-IN: LR-IN1.2, R14.1
- new net N$114: JP5.4, R14.1
- net GND: now also JP5.5, JP5.6; no longer LR-IN1.3, LR-IN1.4
- net N$28: now also JP5.10, JP5.8; no longer JP4.1, LR-IN1.6
- net N$37: now also JP5.7; no longer LR-IN1.5
- net N$52: now also JP5.2; no longer JP2.1
- net N$77: now also JP5.1, JP5.3; no longer JP1.1, LR-IN1.1
- net N$81: now also JP5.9; no longer JP3.1
Other:
- note added: "+ IN = 4 CH 2 : 4-6-8"
- note added: "+ IN = 7 CH 1 : 3-5-7"
- note added: "SJ6 & SJ17 ON : default SJ6 & SJ17 OFF : connect test device to JP5 : 1-2 : CH 1 test JP5 : 9-10 : CH 2 test"
- note removed: "+ IN = 2 CH 2 : 6-4-2"
- note removed: "+ IN = 5 CH 1 : 1-3-5"
- note removed: "SJ6 : JP1-2 & JP3-4 ON : default SJ6 : JP1-2 & JP3-4 open connect test device"
- note removed: "test electrode connection"
- moved on the sheet: SJ17, SJ6
